File: kicad/tab5-fpga-carrier.kicad_pcb (KiCad board)
At the start: 4 copper layers, 125 x 78 mm, 100 parts, among them J1 DC 12-24V, J2 USB-C PD in, J3 M5-BUS (to Tab5), J4 Tang Primer 20K Core, J5 HDMI OUT, J6 PMOD1, J7 PMOD2, J8 GPIO pads, Q1 2N7002, Q2 2N7002, SW1 SW, SW2 RESET (Tab5), SW3 FPGA ON/OFF, U1 CH224K, U2 TPS5430DDAR, U3 AMS1117-3.3, U4 RCLAMP0524P, U5 RCLAMP0524P, U6 SRV05-4

Commit message: Improve D1 TMDS bias routing and independently review PoC suitability
Parts:
- R30, R31: footprint R_0603_1608Metric -> R_0402_1005Metric
- moved R31 8.99 mm to (110.3, 18.2), turned to 0 degrees
- moved R30 8.68 mm to (110.3, 16.8), turned to 0 degrees
Routing:
- net HDMI_D1N_C: track 26.9 -> 16.0 mm, vias 2 -> 0
- net HDMI_D1P_C: track 21.9 -> 16.0 mm, vias 2 -> 0
- net GND: track 124.3 -> 125.7 mm, vias 93 -> 95

Commit message: Prepare PoC parallel isolation, power and manufacturing candidate
Parts:
- added C20: 100n, C_0603_1608Metric, F.Cu at (64.7, 23.5)
- added C21: 100n, C_0603_1608Metric, F.Cu at (64.7, 39.5)
- added C22: 100n, C_0603_1608Metric, F.Cu at (63.0, 65.0)
- added C23: 100n, C_0603_1608Metric, F.Cu at (68.0, 65.0)
- added JP1: BUS ARM (open by default), PinHeader_1x02_P2.54mm_Vertical, F.Cu at (58.9, 71.5)
- added Q3: 2N7002, SOT-23, F.Cu at (63.0, 68.5)
- added Q4: 2N7002, SOT-23, F.Cu at (68.0, 68.5)
- added R46: 22k, R_0603_1608Metric, F.Cu at (68.0, 72.0)
- added R47: 100k, R_0603_1608Metric, F.Cu at (59.5, 65.5)
- added R48: 100k, R_0603_1608Metric, F.Cu at (72.0, 65.0)
- added U10: TPS3839K50DBZR, SOT-23, F.Cu at (68.0, 61.5)
- added U7: SN74CB3Q3245PWR, TSSOP-20_4.4x6.5mm_P0.65mm, F.Cu at (64.7, 28.5)
- added U8: SN74CB3Q3245PWR, TSSOP-20_4.4x6.5mm_P0.65mm, F.Cu at (64.7, 44.5)
- added U9: TPS3839G33DBZR, SOT-23, F.Cu at (63.0, 61.5)
- C7: value 220u/10V polymer -> 220u/10V POSCAP; footprint CP_Elec_6.3x7.7 -> CP_EIA-7343-40_Kemet-Y
- D3: value SMBJ24A (to be selected) -> SMBJ15A
- J1: value DC 12-24V -> DC 12V ONLY
- R7: value 3.3k -> 3.24k
- U3: value AMS1117-3.3 -> TLV1117LV33DCYR
- moved C9 41.5 mm to (48.5, 61.5), turned to 0 degrees
- moved C8 34.0 mm to (45.0, 51.5), turned to 0 degrees
- moved C5 28.6 mm to (39.5, 71.8), turned to 0 degrees
- moved C7 26.9 mm to (39.0, 49.8), turned to 90 degrees
- moved C6 20.1 mm to (33.8, 72.5), turned to 0 degrees
- moved C4 17.7 mm to (33.8, 69.5), turned to 0 degrees
- moved D4 15.9 mm to (27.0, 63.0), turned to 0 degrees
- moved R7 13.0 mm to (20.0, 67.5), turned to 90 degrees
- moved L1 13.0 mm to (39.0, 61.5), turned to 90 degrees
- moved C1 12.2 mm to (27.5, 57.0)
- moved R41 11.4 mm to (50.5, 28.5)
- moved C3 10.2 mm to (22.0, 65.0), turned to 90 degrees
- moved D3 9.18 mm to (18.5, 59.5)
- moved R37 9.00 mm to (59.5, 34.0)
- moved R6 7.43 mm to (22.0, 70.5), turned to 90 degrees
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Connections:
- J4 pad 52: P2_6 -> F_CLK
- J4 pad 80: F_CLK -> P2_6
- R10 pad 1: M_AUX0 -> ISO_CLK
- R10 pad 2: F_AUX0 -> F_CLK
- R11 pad 1: M_RDY -> ISO_AUX0
- R11 pad 2: F_RDY -> F_AUX0
- R12 pad 1: M_D0 -> ISO_RDY
- R12 pad 2: F_D0 -> F_RDY
- R13 pad 1: M_AUX1 -> ISO_D0
- R13 pad 2: F_AUX1 -> F_D0
- R14 pad 1: M_CLK -> ISO_AUX1
- R14 pad 2: F_CLK -> F_AUX1
- R15 pad 1: M_D1 -> ISO_D1
- R16 pad 1: M_D2 -> ISO_D2
- R19 pad 1: M_AUX2 -> ISO_AUX2
- R20 pad 1: M_AUX3 -> ISO_AUX3
- R21 pad 1: M_D4 -> ISO_D4
- R22 pad 1: M_D3 -> ISO_D3
- R23 pad 1: M_D6 -> ISO_D6
- R24 pad 1: M_D5 -> ISO_D5
- R26 pad 1: M_D7 -> ISO_D7
- R27 pad 1: M_DIR -> ISO_DIR
Routing:
- net GND: track 125.7 -> 190.0 mm, vias 95 -> 106
- net BUS_OE_N: track 0.00 -> 53.8 mm, vias 0 -> 2
- net +3V3: track 138.4 -> 187.8 mm, vias 2 -> 6
- net TAB_3V3: track 0.00 -> 36.3 mm
- net +5V: track 174.7 -> 195.3 mm
- net M_EXT37: track 17.3 -> 36.2 mm, vias 0 -> 1
- net BUS_ARM: track 0.00 -> 12.1 mm
- net ISO_CLK: track 0.00 -> 10.7 mm, vias 0 -> 2
- net F_HPD: track 42.5 -> 53.1 mm
- net TAB_PGOOD: track 0.00 -> 10.4 mm, vias 0 -> 1
- net CORE_PGOOD: track 0.00 -> 10.3 mm
- net F_HSDA: track 35.0 -> 45.3 mm
- net ISO_AUX2: track 0.00 -> 9.94 mm, vias 0 -> 2
- net F_CLK: track 29.8 -> 20.3 mm
- net ISO_DIR: track 0.00 -> 9.07 mm, vias 0 -> 2
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