File: kicad/tab5-fpga-carrier.kicad_pcb (KiCad board)
At the start: 4 copper layers, 125 x 78 mm, 114 parts, among them J1 DC 12V ONLY, J2 USB-C PD in, J3 M5-BUS (to Tab5), J4 Tang Primer 20K Core, J5 HDMI OUT, J6 PMOD1, J7 PMOD2, J8 GPIO pads, Q1 2N7002, Q2 2N7002, Q3 2N7002, Q4 2N7002, SW1 SW, SW2 RESET (Tab5), SW3 FPGA ON/OFF, U1 CH224K, U10 TPS3839K50DBZR, U2 TPS5430DDAR, U3 TLV1117LV33DCYR, U4 RCLAMP0524P, U5 RCLAMP0524P, U6 SRV05-4, U7 SN74CB3Q3245PWR, U8 SN74CB3Q3245PWR, U9 TPS3839G33DBZR

Commit message: Correct M5-Bus columns from physical Tab5 confirmation and release PoC files
Parts:
- J3: footprint PinHeader_2x15_P2.54mm_Vertical -> PinHeader_2x15_Tab5_Bottom
Routing:
- net M_AUX0: track 25.1 -> 7.07 mm, vias 1 -> 0
- net M_RDY: track 18.4 -> 6.79 mm
- net M_D0: track 19.0 -> 8.96 mm, vias 2 -> 0
- net PD_VBUS_S: track 11.2 -> 21.0 mm, vias 0 -> 2
- net GND: track 190.0 -> 182.4 mm, vias 106 -> 107
- net F_D1: track 14.6 -> 6.87 mm
- net HDMI_SCL: track 77.2 -> 70.2 mm
- net F_LED2: track 67.8 -> 61.0 mm
- net F_LED0: track 61.8 -> 55.4 mm
- net F_RDY: track 14.0 -> 7.76 mm, vias 2 -> 0
- net PD_CFG3: track 18.0 -> 12.2 mm, vias 3 -> 2
- net BUS_OE_N: track 53.8 -> 59.5 mm, vias 2 -> 4
- net VIN: track 91.3 -> 85.9 mm
- net LED1_A: track 16.0 -> 11.0 mm, vias 2 -> 0
- net M_EXT38: track 14.9 -> 19.4 mm
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