File: kicad/tab5-fpga-carrier.kicad_sch (KiCad schematic)
At the start: 100 parts, among them J1 DC 12-24V, J2 USB-C PD in, J3 M5-BUS (to Tab5), J4 Tang Primer 20K Core, J5 HDMI OUT, J6 PMOD1, J7 PMOD2, J8 GPIO pads, Q1 2N7002, Q2 2N7002, SW1 SW, SW2 RESET (Tab5), SW3 FPGA ON/OFF, U1 CH224K, U2 TPS5430DDAR, U3 AMS1117-3.3, U4 RCLAMP0524P, U5 RCLAMP0524P, U6 SRV05-4

Commit message: Improve D1 TMDS bias routing and independently review PoC suitability
Parts:
- R30, R31: footprint Resistor_SMD:R_0603_1608Metric -> Resistor_SMD:R_0402_1005Metric
Changed lines of the file:
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@@
 			)
 		)
-		(property "Footprint" "Resistor_SMD:R_0603_1608Metric"
+		(property "Footprint" "Resistor_SMD:R_0402_1005Metric"
 			(at 1633.982 314.96 0)
 			(effects
@@
 			)
 		)
-		(property "Footprint" "Resistor_SMD:R_0603_1608Metric"
+		(property "Footprint" "Resistor_SMD:R_0402_1005Metric"
 			(at 1352.042 360.68 0)
 			(effects

Commit message: Prepare PoC parallel isolation, power and manufacturing candidate
Parts:
- added C20, C21, C22, C23: 100n, Capacitor_SMD:C_0603_1608Metric, symbol Device:C
- added JP1: BUS ARM (open by default), Connector_PinHeader_2.54mm:PinHeader_1x02_P2.54mm_Vertical, symbol Connector_Generic:Conn_01x02
- added Q3, Q4: 2N7002, Package_TO_SOT_SMD:SOT-23, symbol Transistor_FET:2N7002
- added R46: 22k, Resistor_SMD:R_0603_1608Metric, symbol Device:R
- added R47, R48: 100k, Resistor_SMD:R_0603_1608Metric, symbol Device:R
- added U10: TPS3839K50DBZR, Package_TO_SOT_SMD:SOT-23, symbol Power_Supervisor:TPS3839DBZ
- added U7, U8: SN74CB3Q3245PWR, Package_SO:TSSOP-20_4.4x6.5mm_P0.65mm, symbol carrier:SN74CB3Q3245
- added U9: TPS3839G33DBZR, Package_TO_SOT_SMD:SOT-23, symbol Power_Supervisor:TPS3839DBZ
- C1: LCSC (none) -> C2983388
- C10, C4, C5: LCSC (none) -> C13585
- C11: LCSC (none) -> C12891
- C12, C13, C14, C15, C16, C17, C18, C19, C6: LCSC (none) -> C14663
- C2: LCSC (none) -> C15849
- C3: LCSC (none) -> C57112
- C7: value 220u/10V polymer -> 220u/10V POSCAP; footprint Capacitor_SMD:CP_Elec_6.3x7.7 -> Capacitor_Tantalum_SMD:CP_EIA-7343-40_Kemet-Y; Comment TI reference design uses 220uF POSCAP on the output (loop c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 -> Panasonic 10TPB220M, 220uF 10V ESR max40mohm; TI reference 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; LCSC (none) -> C242173
- C8, C9: LCSC (none) -> C96123; now not fitted
- D1, D2, D4: LCSC (none) -> C22452
- D3: value SMBJ24A (to be selected) -> SMBJ15A; Comment 24V-class TVS; clamp vs MP4560/TPS5430 abs-max TBD -> YANGJIE 15V standoff, 24.4V specified clamp; regulated 12V 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; LCSC (none) -> C699013
- D5, D6, D7, D8: LCSC (none) -> C2286
- F1: LCSC (none) -> C47002391
- F2: LCSC (none) -> C315893
- J1: value DC 12-24V -> DC 12V ONLY
- J2: LCSC (none) -> C5246813
- L1: LCSC (none) -> C2041333
- Q1, Q2: LCSC (none) -> C8545
- R1, R36, R37, R40, R6: LCSC (none) -> C25804
- R10, R11, R12, R13, R14, R15, R16, R19, R20, R21, R22, R23, R24, R26, R27: LCSC (none) -> C23140
- R17, R18, R25, R3: LCSC (none) -> C21189
- R2, R42, R43, R44, R45: LCSC (none) -> C21190
- R28, R29, R32, R33, R34, R35: LCSC (none) -> C23065
- R30, R31: LCSC (none) -> C4125
- R38, R39: LCSC (none) -> C4190
- R4: Comment CFG3 low (fit) -> 20V; DNP -> 15V -> Must remain DNP: CFG3 internal pull-up for 12V request; LCSC (none) -> C21189; now not fitted
- R41: LCSC (none) -> C4184
- R5: Comment CFG2 low (DNP): fit with CFG3 open -> 12V -> Fitted: CFG2 low, CFG1 low, CFG3 high -> 12V; LCSC (none) -> C21189; now fitted
- R7: value 3.3k -> 3.24k; Comment Vout = 1.221*(1+10k/3.3k) = 4.92V -> Vout = 1.221*(1+10k/3.24k) = 4.99V; R7 C22994 1%; LCSC (none) -> C22994
- R8: LCSC (none) -> C25803
- R9: Comment UVLO ~9.6V (holds off until PD reaches 20V) -> External EN divider ~9.4V threshold; stays off at default U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; LCSC (none) -> C22809
- U1: Comment PD sink, 20V request: CFG1=0 CFG2=1(internal PU) CFG3=0 -> PD sink, 12V request: CFG1=0 CFG2=0 CFG3=1(internal PU); LCSC (none) -> C970725
- U2: LCSC (none) -> C9864
- U3: value AMS1117-3.3 -> TLV1117LV33DCYR; Comment (none) -> TI TLV1117LV33: ceramic-output stable, pin-compatible SOT-2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; LCSC (none) -> C15578
Connections:
- net +3V3: now also C20.1, C21.1, R46.1, U7.20 (VCC), U8.20 (VCC)
- net +5V: now also C23.1, U10.3 (VDD)
- net F_AUX0: now also R11.2; no longer R10.2
- net F_AUX1: now also R14.2; no longer R13.2
- net F_CLK: now also J4.52 (F_CLK), R10.2; no longer J4.80 (F_CLK), R14.2
- net F_D0: now also R13.2; no longer R12.2
- net F_RDY: now also R12.2; no longer R11.2
- net GND: now also C20.2, C21.2, C22.2, C23.2, Q4.2 (S), R47.2, R48.2, U10.1 (GND), U7.10 (GND), U8.10 (GND), U9.1 (GND)
- net M_AUX0: now also U7.3 (A2); no longer R10.1
- net M_AUX1: now also U7.6 (A5); no longer R13.1
- net M_AUX2: now also U7.9 (A8); no longer R19.1
- net M_AUX3: now also U8.2 (A1); no longer R20.1
- net M_CLK: now also U7.2 (A1); no longer R14.1
- net M_D0: now also U7.5 (A4); no longer R12.1
- net M_D1: now also U7.7 (A6); no longer R15.1
- net M_D2: now also U7.8 (A7); no longer R16.1
- net M_D3: now also U8.4 (A3); no longer R22.1
- net M_D4: now also U8.3 (A2); no longer R21.1
- net M_D5: now also U8.6 (A5); no longer R24.1
- net M_D6: now also U8.5 (A4); no longer R23.1
- net M_D7: now also U8.7 (A6); no longer R26.1
- net M_DIR: now also U8.8 (A7); no longer R27.1
- net M_RDY: now also U7.4 (A3); no longer R11.1
- net P2_6: now also J4.80 (P2_6); no longer J4.52 (P2_6)
- net TAB_3V3: now also C22.1, U9.3 (VDD)
- new net BUS_ARM: JP1.2 (Pin_2), Q3.1 (G), R47.1
- new net BUS_OE_MID: Q3.2 (S), Q4.3 (D)
- new net BUS_OE_N: Q3.3 (D), R46.2, U7.19 (~{OE}), U8.19 (~{OE})
- new net CORE_PGOOD: Q4.1 (G), R48.1, U10.2 (~{RESET})
- new net ISO_AUX0: R11.1, U7.17 (B2)
- new net ISO_AUX1: R14.1, U7.14 (B5)
- new net ISO_AUX2: R19.1, U7.11 (B8)
- new net ISO_AUX3: R20.1, U8.18 (B1)
- new net ISO_CLK: R10.1, U7.18 (B1)
- new net ISO_D0: R13.1, U7.15 (B4)
- new net ISO_D1: R15.1, U7.13 (B6)
- new net ISO_D2: R16.1, U7.12 (B7)
- new net ISO_D3: R22.1, U8.16 (B3)
- new net ISO_D4: R21.1, U8.17 (B2)
- new net ISO_D5: R24.1, U8.14 (B5)
- new net ISO_D6: R23.1, U8.15 (B4)
- new net ISO_D7: R26.1, U8.13 (B6)
- new net ISO_DIR: R27.1, U8.12 (B7)
- new net ISO_RDY: R12.1, U7.16 (B3)
- new net TAB_PGOOD: JP1.1 (Pin_1), U9.2 (~{RESET})
- no-connect marks 9 -> 13
Other:
- note added: "Power-off bus isolation + 33R (M=Tab5, ISO=switch, F=FPGA)"
- note added: "USB-C PD sink (CH224K, 12V request)"
- note removed: "33R series resistors (M_* = Tab5 side, F_* = FPGA side)"
- note removed: "USB-C PD sink (CH224K, 20V request)"

Commit message: Correct M5-Bus columns from physical Tab5 confirmation and release PoC files
Parts:
- J3: footprint Connector_PinHeader_2.54mm:PinHeader_2x15_P2.54mm_Vertical -> carrier:PinHeader_2x15_Tab5_Bottom; Comment male header on Tab5-facing side; pin-1 orientation to be co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 -> User confirmed 2026-10-24: rear view, battery left, pin1 GN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
